File: electronics/KiCAD/Realm Card.kicad_pcb (KiCad board)
At the start: 2 copper layers, 50 x 40 mm, 21 parts, among them J1 Conn_02x07_Top_Bottom, J2 Micro_SD_Card, J3 Conn_01x02_Female, J4 Conn_02x25_Top_Bottom, SW1 SW_SPDT, U1 MCP73831-2-OT

Commit message: revised
Parts:
- removed the R4 at (46.5, 29.2)
- added R8: 10K, Resistor_SMD:R_0805_2012Metric, F.Cu at (5.00, 11.5)
- added U2: MCP100-315D, Package_TO_SOT_SMD:SOT-23, F.Cu at (5.00, 8.50)
- D2: value LED GREEN 20 mA @3V -> LED 20 mA @2V
- D3: renamed from D1; value LED RED 10 mA @2V -> LED 20 mA @2V
- R10, R9: value 10K -> 10
- R3: renamed from R5; value 150 -> 68
- R5: renamed from R6; value 100 -> 68
- R6: renamed from R7; value 10K -> 10
- R7: renamed from R8; value 10K -> 10
- moved R10 7.00 mm to (5.00, 13.5)
- moved R6 7.00 mm to (5.00, 19.5)
- moved R7 7.00 mm to (5.00, 17.5)
- moved R9 7.00 mm to (5.00, 15.5)
- moved U1 2.55 mm to (48.0, 27.0)
- renumbered D3 to D1, J3 to J1, J1 to J2, J4 to J3, J2 to J4, R3 to R1, R1 to R2, R2 to R4
Connections:
- J3 pad 10: unconnected-(J4-Pad10) -> reset
- J3 pad 11: Y+ -> unconnected-(J4-Pad11)
- J3 pad 12: X+ -> unconnected-(J4-Pad12)
- J3 pad 13: Y- -> unconnected-(J4-Pad13)
- J3 pad 14: X- -> unconnected-(J4-Pad14)
- J3 pad 44: unconnected-(J4-Pad44) -> X-
- J3 pad 45: unconnected-(J4-Pad45) -> Y-
- J3 pad 46: unconnected-(J4-Pad46) -> X+
- J3 pad 47: unconnected-(J4-Pad47) -> Y+
- J3 pad 6: +3.3V -> GND
- R3 pad 1: Net-(R4-Pad2) -> Net-(R4-Pad1)
Routing:
- net reset: track 0.00 -> 19.5 mm
- net Y+: track 56.1 -> 39.0 mm
- net +3.3V: track 80.7 -> 97.7 mm, vias 7 -> 9
- net Y-: track 59.9 -> 43.8 mm
- net X+: track 51.7 -> 36.2 mm
- net X-: track 55.1 -> 40.8 mm
- net Net-(J4-Pad5): track 11.9 -> 18.0 mm
- net Net-(J4-Pad4): track 12.9 -> 18.6 mm
- net Net-(J4-Pad3): track 13.8 -> 19.3 mm
- net Net-(J4-Pad2): track 14.4 -> 19.9 mm
- net Net-(R3-Pad2): track 9.54 -> 14.8 mm
- net +5V: track 128.0 -> 132.7 mm, vias 8 -> 7
- net SD_CS: track 101.4 -> 105.6 mm
- net BAT CHG: track 29.0 -> 31.5 mm
- net MOSI: track 72.7 -> 74.7 mm
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
Commit message: updated board
Parts:
- added C2: 0.1uf, Capacitor_SMD:C_0805_2012Metric, F.Cu at (42.0, 25.5)
- added R1: 100K, Resistor_SMD:R_0805_2012Metric, F.Cu at (43.0, 15.0)
- added R2: 100K, Resistor_SMD:R_0805_2012Metric, F.Cu at (5.00, 21.5)
- U2: value MCP100-315D -> APX803-44SAG-7
- moved C3 1.00 mm to (42.0, 27.5)
- moved R4 0.96 mm to (43.0, 17.0)
- moved U2 0.56 mm to (4.44, 8.50), turned to 180 degrees
- moved C1 0.50 mm to (42.0, 29.5)
- moved D3 0.50 mm to (41.5, 32.0)
- moved R3 0.42 mm to (43.0, 19.0)
- moved R5 0.13 mm to (43.0, 21.0)
- renumbered C2 to C3, D3 to D1, D1 to D3, J2 to J1, J4 to J2, J1 to J3, J3 to J4, R9 to R10, R10 to R11, R8 to R12, R2 to R3, R1 to R5, R3 to R6, R5 to R7, R7 to R8, R6 to R9
Connections:
- J4 pad 2: Net-(J4-Pad2) -> /LEDA
- J4 pad 3: Net-(J4-Pad3) -> /LEDA
- J4 pad 4: Net-(J4-Pad4) -> /LEDA
- J4 pad 5: Net-(J4-Pad5) -> /LEDA
- R10 pad 2: Net-(J4-Pad4) -> /LEDA
- R11 pad 2: Net-(J4-Pad5) -> /LEDA
- R8 pad 2: Net-(J4-Pad3) -> /LEDA
- R9 pad 2: Net-(J4-Pad2) -> /LEDA
- U2 pad 1: reset -> GND
- U2 pad 2: +3.3V -> reset
- U2 pad 3: GND -> +3.3V
Routing:
- net /LEDA: track 0.00 -> 75.8 mm
- net Net-(J4-Pad2): track 19.9 -> 0.00 mm
- net Net-(J4-Pad3): track 19.3 -> 0.00 mm
- net Net-(J4-Pad4): track 18.6 -> 0.00 mm
- net Net-(J4-Pad5): track 18.0 -> 0.00 mm
- net Y-: track 43.8 -> 50.4 mm
- net +3.3V: track 97.7 -> 103.1 mm, vias 9 -> 11
- net BAT CHG: track 31.5 -> 26.5 mm
- net SD_CS: track 105.6 -> 110.1 mm
- net LCD_CS: track 39.9 -> 44.3 mm, vias 2 -> 6
- net GND: track 4.33 -> 8.71 mm, vias 0 -> 2
- net Net-(J3-Pad1): track 31.3 -> 35.5 mm
- net +5V: track 132.7 -> 128.9 mm, vias 7 -> 6
- net VBAT: track 12.7 -> 16.0 mm
- net X-: track 40.8 -> 39.2 mm
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Other:
- outline, holes or cut-outs redrawn
- board text removed: "QT PY"

Commit message: reworked code
Parts:
- removed U2: APX803-44SAG-7, Package_TO_SOT_SMD:SOT-23
Connections:
- net reset renamed /reset
Routing:
- net +3.3V: track 103.1 -> 101.5 mm, vias 11 -> 10
- net /reset: track 20.5 -> 19.0 mm
Changed lines of the file:
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@@
   (net 48 "unconnected-(J4-Pad13)")
   (net 49 "unconnected-(J4-Pad14)")
-  (net 50 "reset")
+  (net 50 "/reset")
   (footprint "Package_TO_SOT_SMD:SOT-23-5" (layer "F.Cu")
     (at 48 27 -90)
@@
     (fp_line (start -1 0.625) (end -1 -0.625) (layer "F.Fab") (width 0.1))
     (pad "1" smd roundrect (at -0.9125 0 180) (size 1.025 1.4) (layers "F.Cu" "F.Paste" "F.Mask") (roundrect_rratio 0.243902439)
-      (net 50 "reset") (pintype "passive"))
+      (net 50 "/reset") (pintype "passive"))
     (pad "2" smd roundrect (at 0.9125 0 180) (size 1.025 1.4) (layers "F.Cu" "F.Paste" "F.Mask") (roundrect_rratio 0.243902439)
       (net 6 "+3.3V") (pintype "passive"))
@@
       (net 6 "+3.3V") (pinfunction "Pin_9") (pintype "passive"))
     (pad "10" smd rect (at -7.75 -1.85) (size 0.3 1.3) (layers "F.Cu" "F.Paste" "F.Mask")
-      (net 50 "reset") (pinfunction "Pin_10") (pintype "passive"))
+      (net 50 "/reset") (pinfunction "Pin_10") (pintype "passive"))
     (pad "11" smd rect (at -7.25 -1.85) (size 0.3 1.3) (layers "F.Cu" "F.Paste" "F.Mask")
       (net 46 "unconnected-(J4-Pad11)") (pinfunction "Pin_11") (pintype "passive+no_connect"))
@@
     )
   )
-  (footprint "Package_TO_SOT_SMD:SOT-23" (layer "F.Cu")
-    (at 4.4375 8.5 180)
-    (descr "SOT, 3 Pin (https://www.jedec.org/system/files/docs/to-236h.pdf variant AB), generated with kicad-footprint-generator ipc_gullwing_generator.py")
-    (tags "SOT TO_SOT_SMD")
-    (property "LCSC" "C155243")
-    (property "Sheetfile" "Realm Card.kicad_sch")
-    (property "Sheetname" "")
-    (attr smd)
-    (fp_text reference "U2" (at 3 0) (layer "F.SilkS")
-      (effects (font (size 1 1) (thickness 0.15)))
-    )
-    (fp_text value "APX803-44SAG-7" (at 0 2.4) (layer "F.Fab")
-      (effects (font (size 1 1) (thickness 0.15)))
-    )
-    (fp_text user "${REFERENCE}" (at 0 0) (layer "F.Fab")
-      (effects (font (size 0.32 0.32) (thickness 0.05)))
-    )
-    (fp_line (start 0 -1.56) (end 0.65 -1.56) (layer "F.SilkS") (width 0.12))
-    (fp_line (start 0 1.56) (end -0.65 1.56) (layer "F.SilkS") (width 0.12))
-    (fp_line (start 0 -1.56) (end -1.675 -1.56) (layer "F.SilkS") (width 0.12))
-    (fp_line (start 0 1.56) (end 0.65 1.56) (layer "F.SilkS") (width 0.12))
-    (fp_line (start 1.92 -1.7) (end -1.92 -1.7) (layer "F.CrtYd") (width 0.05))
-    (fp_line (start -1.92 1.7) (end 1.92 1.7) (layer "F.CrtYd") (width 0.05))
-    (fp_line (start 1.92 1.7) (end 1.92 -1.7) (layer "F.CrtYd") (width 0.05))
-    (fp_line (start -1.92 -1.7) (end -1.92 1.7) (layer "F.CrtYd") (width 0.05))
-    (fp_line (start -0.65 1.45) (end -0.65 -1.125) (layer "F.Fab") (width 0.1))
-    (fp_line (start -0.65 -1.125) (end -0.325 -1.45) (layer "F.Fab") (width 0.1))
-    (fp_line (start 0.65 -1.45) (end 0.65 1.45) (layer "F.Fab") (width 0.1))
-    (fp_line (start 0.65 1.45) (end -0.65 1.45) (layer "F.Fab") (width 0.1))
-    (fp_line (start -0.325 -1.45) (end 0.65 -1.45) (layer "F.Fab") (width 0.1))
-    (pad "1" smd roundrect (at -0.9375 -0.95 180) (size 1.475 0.6) (layers "F.Cu" "F.Paste" "F.Mask") (roundrect_rratio 0.25)
-      (net 1 "GND") (pinfunction "GND") (pintype "power_in"))
-    (pad "2" smd roundrect (at -0.9375 0.95 180) (size 1.475 0.6) (layers "F.Cu" "F.Paste" "F.Mask") (roundrect_rratio 0.25)
-      (net 50 "reset") (pinfunction "~{RESET}") (pintype "output"))
-    (pad "3" smd roundrect (at 0.9375 0 180) (size 1.475 0.6) (layers "F.Cu" "F.Paste" "F.Mask") (roundrect_rratio 0.25)
-      (net 6 "+3.3V") (pinfunction "VCC") (pintype "power_in"))
-    (model "${KICAD6_3DMODEL_DIR}/Package_TO_SOT_SMD.3dshapes/SOT-23.wrl"
-      (offset (xyz 0 0 0))
-      (scale (xyz 1 1 1))
-      (rotate (xyz 0 0 0))
-    )
-  )
   (gr_poly
     (pts
@@
   (segment (start 32.25 7.44) (end 32.25 6.49) (width 0.25) (layer "F.Cu") (net 6))
   (segment (start 16.424975 7.924975) (end 17.369027 8.869027) (width 0.25) (layer "F.Cu") (net 6))
-  (segment (start 3.5 7.549904) (end 2.987452 7.037356) (width 0.25) (layer "F.Cu") (net 6))
   (segment (start 5.619301 30.119301) (end 9.012299 33.512299) (width 0.25) (layer "F.Cu") (net 6))
   (segment (start 32.75 6.49) (end 32.25 6.49) (width 0.25) (layer "F.Cu") (net 6))
@@
   (segment (start 6.805 35.669695) (end 8.962396 33.512299) (width 0.25) (layer "F.Cu") (net 6))
   (segment (start 40.7755 15) (end 42.05 15) (width 0.25) (layer "F.Cu") (net 6))
-  (segment (start 3.5 8.5) (end 3.5 7.549904) (width 0.25) (layer "F.Cu") (net 6))
   (segment (start 17.38 32.54) (end 13.54 32.54) (width 0.25) (layer "F.Cu") (net 6))
   (segment (start 16.75 6.49) (end 16.25 6.49) (width 0.25) (layer "F.Cu") (net 6))
@@
   (via (at 32.5 9.5) (size 0.8) (drill 0.4) (layers "F.Cu" "B.Cu") (net 6))
   (via (at 31 8.2755) (size 0.8) (drill 0.4) (layers "F.Cu" "B.Cu") (net 6))
-  (via (at 2.987452 7.037356) (size 0.8) (drill 0.4) (layers "F.Cu" "B.Cu") (net 6))
   (via (at 5.619301 26.8561) (size 0.8) (drill 0.4) (layers "F.Cu" "B.Cu") (net 6))
   (via (at 9.012299 33.512299) (size 0.8) (drill 0.4) (layers "F.Cu" "B.Cu") (net 6))
@@
   (segment (start 17.25 5.54) (end 15.26 3.55) (width 0.25) (layer "F.Cu") (net 50))
   (segment (start 8.391916 4.5625) (end 7.5 5.454416) (width 0.25) (layer "F.Cu") (net 50))
-  (segment (start 5.375 7.55) (end 6.8625 7.55) (width 0.25) (layer "F.Cu") (net 50))
   (segment (start 9.404416 3.55) (end 8.391916 4.5625) (width 0.25) (layer "F.Cu") (net 50))
   (segment (start 15.26 3.55) (end 9.404416 3.55) (width 0.25) (layer "F.Cu") (net 50))

Commit message: Added documentation
Parts:
- removed D2: LED 20 mA @2V, LED_SMD:LED_0805_2012Metric
- removed R7: 68, Resistor_SMD:R_0805_2012Metric
Routing:
- net Net-(R6-Pad1): track 9.91 -> 7.38 mm
- net Net-(D2-Pad2): track 2.02 -> 0.00 mm
Other:
- outline, holes or cut-outs redrawn
- board text added: "REV. C"
- board text removed: "DN"
- board text removed: "REV. B"
