File: electronics/KiCAD/Realm Card.kicad_sch (KiCad schematic)
At the start: 21 parts, among them J1 Conn_02x07_Top_Bottom, J2 Micro_SD_Card, J3 Conn_01x02_Female, J4 Conn_02x25_Top_Bottom, SW1 SW_SPDT, U1 MCP73831-2-OT

Commit message: revised
Parts:
- removed R4: 150, Resistor_SMD:R_0805_2012Metric, symbol Device:R
- added R8: 10K, Resistor_SMD:R_0805_2012Metric, symbol Device:R
- added U2: MCP100-315D, Package_TO_SOT_SMD:SOT-23, symbol Power_Supervisor:MCP100-315D
- D1: value LED RED 10 mA @2V -> LED 20 mA @2V; LCSC C497942 -> C2296
- D2: value LED GREEN 20 mA @3V -> LED 20 mA @2V; LCSC C497948 -> C2296
- R10, R9: value 10K -> 10
- R4: renamed from R5; value 150 -> 68
- R5: renamed from R6; value 100 -> 68
- R6: renamed from R7; value 10K -> 10
- R7: renamed from R8; value 10K -> 10
Connections:
- net +3.3V: now also R8.2, U2.2 (VDD); no longer J4.6 (Pin_6)
- net GND: now also J4.6 (Pin_6), U2.3 (VSS)
- net X+: now also J4.46 (Pin_46); no longer J4.12 (Pin_12)
- net X-: now also J4.44 (Pin_44); no longer J4.14 (Pin_14)
- net Y+: now also J4.47 (Pin_47); no longer J4.11 (Pin_11)
- net Y-: now also J4.45 (Pin_45); no longer J4.13 (Pin_13)
- net LEDA: now reaches J4.2 (Pin_2), R6.2
- net LEDA: now also J4.3 (Pin_3), J4.4 (Pin_4), J4.5 (Pin_5), R10.2, R7.2, R9.2
- net reset: now reaches J4.10 (Pin_10)
- net reset: now also R8.1, U2.1 (~{RST})
- net at R4.1: now also R5.1, U1.1 (STAT)
- no-connect marks 28 -> 27
Other:
- moved on the sheet: D1, D2, R4

Commit message: updated board
Parts:
- removed U2: MCP100-315D, Package_TO_SOT_SMD:SOT-23, symbol Power_Supervisor:MCP100-315D
- added C2: 0.1uf, Capacitor_SMD:C_0805_2012Metric, symbol Device:C
- added R1, R2: 100K, Resistor_SMD:R_0805_2012Metric, symbol Device:R
- added U2: APX803-44SAG-7, Package_TO_SOT_SMD:SOT-23, symbol Power_Supervisor:LM809
- renumbered C2 to C3, R7 to R10, R6 to R11, R8 to R12, R1 to R3, R2 to R4, R3 to R5, R4 to R6, R5 to R7, R10 to R8
Connections:
- net +3.3V: now also R1.2, R2.1, U2.3 (VCC)
- net GND: now also C2.1, U2.1 (GND)
- net LCD_CS: now also R1.1
- net SD_CS: now also R2.2
- net VBAT: now also C2.2
- net reset: now also U2.2 (~{RESET})
Other:
- moved on the sheet: C1, C3, D1, D2, D3, J1, J2, J3, J4, R10, R11, R12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

Commit message: revised code
Parts:
- U2: LCSC C155243 -> C9965
Changed lines of the file:
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@@
       (effects (font (size 1.27 1.27)) hide)
     )
-    (property "LCSC" "C155243" (id 5) (at 118.11 134.62 0)
+    (property "LCSC" "C9965" (id 5) (at 118.11 134.62 0)
       (effects (font (size 1.27 1.27)) hide)
     )

Commit message: reworked code
Parts:
- removed U2: APX803-44SAG-7, Package_TO_SOT_SMD:SOT-23, symbol Power_Supervisor:LM809
Other:
- moved on the sheet: R12
Changed lines of the file:
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@@
   (junction (at 59.69 140.97) (diameter 0) (color 0 0 0 0)
-  )
-  (junction (at 132.08 134.62) (diameter 0) (color 0 0 0 0)
   )
   (junction (at 59.69 143.51) (diameter 0) (color 0 0 0 0)
@@
     (stroke (width 0) (type default) (color 0 0 0 0))
   )
-  (wire (pts (xy 132.08 123.19) (xy 132.08 125.73))
-    (stroke (width 0) (type default) (color 0 0 0 0))
-  )
-  (wire (pts (xy 132.08 134.62) (xy 132.08 133.35))
-    (stroke (width 0) (type default) (color 0 0 0 0))
-  )
   (wire (pts (xy 41.91 115.57) (xy 44.45 115.57))
     (stroke (width 0) (type default) (color 0 0 0 0))
@@
     (stroke (width 0) (type default) (color 0 0 0 0))
   )
+  (wire (pts (xy 41.91 128.27) (xy 44.45 128.27))
+    (stroke (width 0) (type default) (color 0 0 0 0))
+  )
   (wire (pts (xy 35.56 107.95) (xy 44.45 107.95))
     (stroke (width 0) (type default) (color 0 0 0 0))
@@
     (stroke (width 0) (type default) (color 0 0 0 0))
   )
-  (wire (pts (xy 40.64 128.27) (xy 44.45 128.27))
-    (stroke (width 0) (type default) (color 0 0 0 0))
-  )
   (wire (pts (xy 82.55 21.59) (xy 82.55 22.86))
     (stroke (width 0) (type default) (color 0 0 0 0))
@@
     (stroke (width 0) (type default) (color 0 0 0 0))
   )
-  (wire (pts (xy 118.11 121.92) (xy 118.11 124.46))
-    (stroke (width 0) (type default) (color 0 0 0 0))
-  )
   (wire (pts (xy 57.15 166.37) (xy 59.69 166.37))
     (stroke (width 0) (type default) (color 0 0 0 0))
@@
     (stroke (width 0) (type default) (color 0 0 0 0))
   )
-  (wire (pts (xy 132.08 134.62) (xy 133.35 134.62))
-    (stroke (width 0) (type default) (color 0 0 0 0))
-  )
   (wire (pts (xy 102.87 54.61) (xy 105.41 54.61))
     (stroke (width 0) (type default) (color 0 0 0 0))
@@
     (stroke (width 0) (type default) (color 0 0 0 0))
   )
-  (wire (pts (xy 118.11 144.78) (xy 118.11 147.32))
-    (stroke (width 0) (type default) (color 0 0 0 0))
-  )
   (wire (pts (xy 59.69 143.51) (xy 59.69 146.05))
     (stroke (width 0) (type default) (color 0 0 0 0))
@@
     (stroke (width 0) (type default) (color 0 0 0 0))
   )
+  (wire (pts (xy 31.75 128.27) (xy 34.29 128.27))
+    (stroke (width 0) (type default) (color 0 0 0 0))
+  )
   (wire (pts (xy 97.79 91.44) (xy 102.87 91.44))
     (stroke (width 0) (type default) (color 0 0 0 0))
@@
   )
   (wire (pts (xy 118.11 91.44) (xy 127 91.44))
-    (stroke (width 0) (type default) (color 0 0 0 0))
-  )
-  (wire (pts (xy 125.73 134.62) (xy 132.08 134.62))
     (stroke (width 0) (type default) (color 0 0 0 0))
   )
@@
     (property "Intersheet References" "${INTERSHEET_REFS}" (id 0) (at 64.8245 130.8894 0)
       (effects (font (size 1.27 1.27)) (justify left) hide)
-    )
-  )
-  (global_label "reset" (shape input) (at 40.64 128.27 180) (fields_autoplaced)
-    (effects (font (size 1.27 1.27)) (justify right))
-    (property "Intersheet References" "${INTERSHEET_REFS}" (id 0) (at 33.5098 128.3494 0)
-      (effects (font (size 1.27 1.27)) (justify right) hide)
     )
   )
@@
     )
   )
-  (global_label "reset" (shape input) (at 133.35 134.62 0) (fields_autoplaced)
-    (effects (font (size 1.27 1.27)) (justify left))
-    (property "Intersheet References" "${INTERSHEET_REFS}" (id 0) (at 140.4802 134.5406 0)
-      (effects (font (size 1.27 1.27)) (justify left) hide)
-    )
-  )
   (symbol (lib_id "Device:R") (at 38.1 115.57 90) (unit 1)
     (in_bom yes) (on_board yes)
@@
     (pin "1")
     (pin "2")
-  )
-  (symbol (lib_id "power:GND") (at 118.11 147.32 0) (unit 1)
-    (in_bom yes) (on_board yes)
-    (property "Reference" "#PWR028" (id 0) (at 118.11 153.67 0)
-      (effects (font (size 1.27 1.27)) hide)
-    )
-    (property "Value" "GND" (id 1) (at 115.57 151.13 0)
-      (effects (font (size 1.27 1.27)) (justify left))
-    )
-    (property "Footprint" "" (id 2) (at 118.11 147.32 0)
-      (effects (font (size 1.27 1.27)) hide)
-    )
-    (property "Datasheet" "" (id 3) (at 118.11 147.32 0)
-      (effects (font (size 1.27 1.27)) hide)
-    )
-    (pin "1")
-  )
-  (symbol (lib_id "Power_Supervisor:LM809") (at 118.11 134.62 0) (unit 1)
-    (in_bom yes) (on_board yes) (fields_autoplaced)
-    (property "Reference" "U2" (id 0) (at 111.76 133.3499 0)
-      (effects (font (size 1.27 1.27)) (justify right))
-    )
-    (property "Value" "APX803-44SAG-7" (id 1) (at 111.76 135.8899 0)
-      (effects (font (size 1.27 1.27)) (justify right))
-    )
-    (property "Footprint" "Package_TO_SOT_SMD:SOT-23" (id 2) (at 125.73 132.08 0)
-      (effects (font (size 1.27 1.27)) hide)
-    )
-    (property "Datasheet" "http://www.ti.com/lit/ds/symlink/lm809.pdf" (id 3) (at 125.73 132.08 0)
-      (effects (font (size 1.27 1.27)) hide)
-    )
-    (property "LCSC" "C9965" (id 5) (at 118.11 134.62 0)
-      (effects (font (size 1.27 1.27)) hide)
-    )
-    (pin "1")
-    (pin "2")
-    (pin "3")
   )
   (symbol (lib_id "Connector:Micro_SD_Card") (at 52.07 74.93 0) (unit 1)
@@
     (pin "1")
   )
-  (symbol (lib_id "power:+3.3V") (at 118.11 121.92 0) (unit 1)
-    (in_bom yes) (on_board yes) (fields_autoplaced)
-    (property "Reference" "#PWR024" (id 0) (at 118.11 125.73 0)
-      (effects (font (size 1.27 1.27)) hide)
-    )
-    (property "Value" "+3.3V" (id 1) (at 120.65 120.6499 0)
-      (effects (font (size 1.27 1.27)) (justify left))
-    )
-    (property "Footprint" "" (id 2) (at 118.11 121.92 0)
-      (effects (font (size 1.27 1.27)) hide)
-    )
-    (property "Datasheet" "" (id 3) (at 118.11 121.92 0)
-      (effects (font (size 1.27 1.27)) hide)
-    )
-    (pin "1")
-  )
   (symbol (lib_id "power:+3.3V") (at 82.55 41.91 180) (unit 1)
     (in_bom yes) (on_board yes) (fields_autoplaced)
@@
     (pin "1")
   )
-  (symbol (lib_id "Device:R") (at 132.08 129.54 180) (unit 1)
-    (in_bom yes) (on_board yes)
-    (property "Reference" "R12" (id 0) (at 129.54 129.54 90))
-    (property "Value" "10K" (id 1) (at 132.08 129.54 90))
-    (property "Footprint" "Resistor_SMD:R_0805_2012Metric" (id 2) (at 133.858 129.54 90)
-      (effects (font (size 1.27 1.27)) hide)
-    )
-    (property "Datasheet" "~" (id 3) (at 132.08 129.54 0)
+  (symbol (lib_id "Device:R") (at 38.1 128.27 270) (unit 1)
+    (in_bom yes) (on_board yes)
+    (property "Reference" "R12" (id 0) (at 38.1 130.81 90))
+    (property "Value" "10K" (id 1) (at 38.1 128.27 90))
+    (property "Footprint" "Resistor_SMD:R_0805_2012Metric" (id 2) (at 38.1 126.492 90)
+      (effects (font (size 1.27 1.27)) hide)
+    )
+    (property "Datasheet" "~" (id 3) (at 38.1 128.27 0)
       (effects (font (size 1.27 1.27)) hide)
     )
@@
     )
     (property "Datasheet" "" (id 3) (at 127 101.6 0)
+      (effects (font (size 1.27 1.27)) hide)
+    )
+    (pin "1")
+  )
+  (symbol (lib_id "power:+3.3V") (at 31.75 128.27 90) (unit 1)
+    (in_bom yes) (on_board yes) (fields_autoplaced)
+    (property "Reference" "#PWR?" (id 0) (at 35.56 128.27 0)
+      (effects (font (size 1.27 1.27)) hide)
+    )
+    (property "Value" "+3.3V" (id 1) (at 27.94 128.2699 90)
+      (effects (font (size 1.27 1.27)) (justify left))
+    )
+    (property "Footprint" "" (id 2) (at 31.75 128.27 0)
+      (effects (font (size 1.27 1.27)) hide)
+    )
+    (property "Datasheet" "" (id 3) (at 31.75 128.27 0)
       (effects (font (size 1.27 1.27)) hide)
     )
@@
     (pin "1")
   )
-  (symbol (lib_id "power:+3.3V") (at 132.08 123.19 0) (unit 1)
-    (in_bom yes) (on_board yes) (fields_autoplaced)
-    (property "Reference" "#PWR025" (id 0) (at 132.08 127 0)
-      (effects (font (size 1.27 1.27)) hide)
-    )
-    (property "Value" "+3.3V" (id 1) (at 134.62 121.9199 0)
-      (effects (font (size 1.27 1.27)) (justify left))
-    )
-    (property "Footprint" "" (id 2) (at 132.08 123.19 0)
-      (effects (font (size 1.27 1.27)) hide)
-    )
-    (property "Datasheet" "" (id 3) (at 132.08 123.19 0)
-      (effects (font (size 1.27 1.27)) hide)
-    )
-    (pin "1")
-  )
   (symbol (lib_id "Device:R") (at 31.75 113.03 90) (unit 1)
     (in_bom yes) (on_board yes)
@@
       (reference "#PWR023") (unit 1) (value "+3.3V") (footprint "")
     )
-    (path "/8e404ad0-986c-4a85-9e19-189e3f43b749"
-      (reference "#PWR024") (unit 1) (value "+3.3V") (footprint "")
-    )
-    (path "/df85079f-08cc-46e4-b3d3-d1827057fc72"
-      (reference "#PWR025") (unit 1) (value "+3.3V") (footprint "")
-    )
     (path "/a57d186d-c44c-488e-adf9-29d1f7920d84"
       (reference "#PWR026") (unit 1) (value "+3.3V") (footprint "")
@@
       (reference "#PWR027") (unit 1) (value "GND") (footprint "")
     )
-    (path "/0c1d656a-0cba-4523-8468-c4916ff160c8"
-      (reference "#PWR028") (unit 1) (value "GND") (footprint "")
-    )
     (path "/616bab85-976f-4cfb-92dd-725aad841618"
       (reference "#PWR029") (unit 1) (value "GND") (footprint "")
     )
+    (path "/dc6fa591-0f2d-4bb4-8614-cfcfcd4bdd12"
+      (reference "#PWR?") (unit 1) (value "+3.3V") (footprint "")
+    )
     (path "/2d810b3f-a880-4019-a0af-6c641e7e04df"
       (reference "C1") (unit 1) (value "10uF") (footprint "Capacitor_SMD:C_0805_2012Metric")
@@
       (reference "U1") (unit 1) (value "MCP73831-2-OT") (footprint "Package_TO_SOT_SMD:SOT-23-5")
     )
-    (path "/1e23b608-0799-41bc-a2a4-f859cca34eb2"
-      (reference "U2") (unit 1) (value "APX803-44SAG-7") (footprint "Package_TO_SOT_SMD:SOT-23")
-    )
-  )
+  )

Commit message: Added documentation
Parts:
- removed D2: LED 20 mA @2V, LED_SMD:LED_0805_2012Metric, symbol Device:LED
- removed R7: 68, Resistor_SMD:R_0805_2012Metric, symbol Device:R
Changed lines of the file:
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@@
   (junction (at 25.4 113.03) (diameter 0) (color 0 0 0 0)
-  )
-  (junction (at 132.08 54.61) (diameter 0) (color 0 0 0 0)
   )
   (junction (at 59.69 163.83) (diameter 0) (color 0 0 0 0)
@@
     (stroke (width 0) (type default) (color 0 0 0 0))
   )
-  (wire (pts (xy 125.73 54.61) (xy 132.08 54.61))
+  (wire (pts (xy 125.73 54.61) (xy 133.35 54.61))
     (stroke (width 0) (type default) (color 0 0 0 0))
   )
@@
     (stroke (width 0) (type default) (color 0 0 0 0))
   )
-  (wire (pts (xy 148.59 64.77) (xy 151.13 64.77))
-    (stroke (width 0) (type default) (color 0 0 0 0))
-  )
   (wire (pts (xy 57.15 135.89) (xy 59.69 135.89))
     (stroke (width 0) (type default) (color 0 0 0 0))
@@
     (stroke (width 0) (type default) (color 0 0 0 0))
   )
-  (wire (pts (xy 132.08 54.61) (xy 132.08 64.77))
-    (stroke (width 0) (type default) (color 0 0 0 0))
-  )
   (wire (pts (xy 26.67 72.39) (xy 29.21 72.39))
     (stroke (width 0) (type default) (color 0 0 0 0))
@@
     (stroke (width 0) (type default) (color 0 0 0 0))
   )
-  (wire (pts (xy 139.7 64.77) (xy 140.97 64.77))
-    (stroke (width 0) (type default) (color 0 0 0 0))
-  )
   (wire (pts (xy 57.15 133.35) (xy 59.69 133.35))
     (stroke (width 0) (type default) (color 0 0 0 0))
@@
   )
   (wire (pts (xy 57.15 123.19) (xy 59.69 123.19))
-    (stroke (width 0) (type default) (color 0 0 0 0))
-  )
-  (wire (pts (xy 132.08 54.61) (xy 133.35 54.61))
     (stroke (width 0) (type default) (color 0 0 0 0))
   )
@@
     (pin "1")
   )
-  (symbol (lib_id "Device:R") (at 135.89 64.77 90) (unit 1)
-    (in_bom yes) (on_board yes)
-    (property "Reference" "R7" (id 0) (at 135.89 62.23 90))
-    (property "Value" "68" (id 1) (at 135.89 64.77 90))
-    (property "Footprint" "Resistor_SMD:R_0805_2012Metric" (id 2) (at 135.89 66.548 90)
-      (effects (font (size 1.27 1.27)) hide)
-    )
-    (property "Datasheet" "~" (id 3) (at 135.89 64.77 0)
-      (effects (font (size 1.27 1.27)) hide)
-    )
-    (pin "1")
-    (pin "2")
-  )
   (symbol (lib_id "Battery_Management:MCP73831-2-OT") (at 115.57 52.07 0) (unit 1)
     (in_bom yes) (on_board yes) (fields_autoplaced)
@@
     (pin "5")
   )
-  (symbol (lib_id "power:GND") (at 151.13 64.77 90) (unit 1)
-    (in_bom yes) (on_board yes) (fields_autoplaced)
-    (property "Reference" "#PWR011" (id 0) (at 157.48 64.77 0)
-      (effects (font (size 1.27 1.27)) hide)
-    )
-    (property "Value" "GND" (id 1) (at 154.94 64.7699 90)
-      (effects (font (size 1.27 1.27)) (justify right))
-    )
-    (property "Footprint" "" (id 2) (at 151.13 64.77 0)
-      (effects (font (size 1.27 1.27)) hide)
-    )
-    (property "Datasheet" "" (id 3) (at 151.13 64.77 0)
-      (effects (font (size 1.27 1.27)) hide)
-    )
-    (pin "1")
-  )
   (symbol (lib_id "power:GND") (at 132.08 36.83 270) (unit 1)
     (in_bom yes) (on_board yes)
@@
     )
     (pin "1")
-  )
-  (symbol (lib_id "Device:LED") (at 144.78 64.77 180) (unit 1)
-    (in_bom yes) (on_board yes)
-    (property "Reference" "D2" (id 0) (at 144.78 62.23 0))
-    (property "Value" "LED 20 mA @2V" (id 1) (at 144.78 67.31 0))
-    (property "Footprint" "LED_SMD:LED_0805_2012Metric" (id 2) (at 144.78 64.77 0)
-      (effects (font (size 1.27 1.27)) hide)
-    )
-    (property "Datasheet" "~" (id 3) (at 144.78 64.77 0)
-      (effects (font (size 1.27 1.27)) hide)
-    )
-    (property "LCSC" "C2296" (id 4) (at 144.78 64.77 0)
-      (effects (font (size 1.27 1.27)) hide)
-    )
-    (pin "1")
-    (pin "2")
   )
   (symbol (lib_id "Device:R") (at 82.55 26.67 180) (unit 1)
@@
   (symbol (lib_id "power:+3.3V") (at 31.75 128.27 90) (unit 1)
     (in_bom yes) (on_board yes) (fields_autoplaced)
-    (property "Reference" "#PWR?" (id 0) (at 35.56 128.27 0)
+    (property "Reference" "#PWR0101" (id 0) (at 35.56 128.27 0)
       (effects (font (size 1.27 1.27)) hide)
     )
@@
       (reference "#PWR010") (unit 1) (value "+5V") (footprint "")
     )
-    (path "/b6feb332-758c-4d3f-a9c9-06834fac6f39"
-      (reference "#PWR011") (unit 1) (value "GND") (footprint "")
-    )
     (path "/e6f90d97-ba38-410d-8e5a-eaa1cbb9714a"
       (reference "#PWR012") (unit 1) (value "+5V") (footprint "")
@@
     )
     (path "/dc6fa591-0f2d-4bb4-8614-cfcfcd4bdd12"
-      (reference "#PWR?") (unit 1) (value "+3.3V") (footprint "")
+      (reference "#PWR0101") (unit 1) (value "+3.3V") (footprint "")
     )
     (path "/2d810b3f-a880-4019-a0af-6c641e7e04df"
@@
       (reference "D1") (unit 1) (value "LED 20 mA @2V") (footprint "LED_SMD:LED_0805_2012Metric")
     )
-    (path "/bb552f03-aaa8-4fa9-9615-fcb7eb719b5f"
-      (reference "D2") (unit 1) (value "LED 20 mA @2V") (footprint "LED_SMD:LED_0805_2012Metric")
-    )
     (path "/5fd5a77b-1dd0-4670-a3cd-72fd3acca386"
       (reference "D3") (unit 1) (value "20V 1A") (footprint "Diode_SMD:D_SOD-123")
@@
       (reference "R6") (unit 1) (value "68") (footprint "Resistor_SMD:R_0805_2012Metric")
     )
-    (path "/a5a023c3-4c16-409e-b903-b3e3b8bc5f55"
-      (reference "R7") (unit 1) (value "68") (footprint "Resistor_SMD:R_0805_2012Metric")
-    )
     (path "/6a2e943f-6559-4376-8af2-d5a7da9aefa3"
